File: kicad/Project Helena.kicad_pcb (KiCad board)
At the start: 2 copper layers, 346 x 111 mm, 68 parts, among them J1 Conn_01x24, J2 Conn_01x08, J3 Conn_01x08, SW1 BREAK, SW10 H, SW11 SPACE, SW12 HELP, SW13 8, SW14 5, SW15 I, SW16 T, SW17 K, SW18 G, SW19 M, SW2 CONTROL, SW20 B, SW21 START, SW22 9, SW23 4, SW24 O, SW25 R, SW26 L, SW27 F, SW28 COMMA, SW29 V, SW3 SHIFT_L, SW30 SELECT, SW31 0, SW32 3, SW33 P, SW34 E, SW35 SEMICOLON, SW36 D, SW37 PERIOD, SW38 C, SW39 OPTION, SW4 7, SW40 <, SW41 2, SW42 MINUS, SW43 W, SW44 PLUS, SW45 S, SW46 SLASH, SW47 X, SW48 RESET, SW49 >, SW5 6, SW50 1, SW51 EQUAL, SW52 Q, SW53 ASTERISK, SW54 A, SW55 INV, SW56 Z, SW57 DEL, SW58 ESC, SW59 RETURN, SW6 U, SW60 TAB, SW61 CAPS, SW62 SPACE, SW63 SPACE, SW64 SHIFT_R, SW7 Y, SW8 N, SW9 J

Commit message: Created Rev B
Rev B of ivops Atari600xl keyboard.
Modified switch footprints to accommodate 5 holes for stability. 
Added PCB mount stabilizer holes for 3D printed brackets.
Added through-holes to match the metal backplate on my membrane 600xl keyboard with the intention of making stand-offs.
Extensively rerouted traces to avoid all the new holes.
Parts:
- removed SW62, SW63: SPACE, Button_Switch_Keyboard:SW_Cherry_MX1A_1.00u_Plate
- added REF01: MountingHole_2.5mm, MountingHole:MountingHole_2.5mm, F.Cu at (50.7, 77.7)
- added REF02: MountingHole_2.5mm, MountingHole:MountingHole_2.5mm, F.Cu at (129.3, 77.7)
- added REF03: MountingHole_2.5mm, MountingHole:MountingHole_2.5mm, F.Cu at (205.5, 77.7)
- added REF04: MountingHole_2.5mm, MountingHole:MountingHole_2.5mm, F.Cu at (262.7, 77.7)
- added REF05: MountingHole_2.5mm, MountingHole:MountingHole_2.5mm, F.Cu at (319.8, 77.7)
- added REF06: MountingHole_2.5mm, MountingHole:MountingHole_2.5mm, F.Cu at (40.7, 111.6)
- added REF07: MountingHole_2.5mm, MountingHole:MountingHole_2.5mm, F.Cu at (181.2, 111.6)
- added REF08: MountingHole_2.5mm, MountingHole:MountingHole_2.5mm, F.Cu at (276.4, 111.6)
- added REF09: MountingHole_2.5mm, MountingHole:MountingHole_2.5mm, F.Cu at (317.6, 115.8)
- added REF10: MountingHole_2.5mm, MountingHole:MountingHole_2.5mm, F.Cu at (128.7, 130.6)
- added REF11: MountingHole_2.5mm, MountingHole:MountingHole_2.5mm, F.Cu at (47.7, 149.7)
- added REF12: MountingHole_2.5mm, MountingHole:MountingHole_2.5mm, F.Cu at (182.1, 153.9)
- added REF13: MountingHole_2.5mm, MountingHole:MountingHole_2.5mm, F.Cu at (233.7, 149.7)
- added REF14: MountingHole_2.5mm, MountingHole:MountingHole_2.5mm, F.Cu at (305.1, 149.7)
- added REF15: MountingHole_2.5mm, MountingHole:MountingHole_2.5mm, F.Cu at (342.5, 77.7)
- added REF16: MountingHole_2.5mm, MountingHole:MountingHole_2.5mm, F.Cu at (357.3, 130.6)
- added REF17: MountingHole_2.5mm, MountingHole:MountingHole_2.5mm, F.Cu at (342.5, 153.9)
- added REF18: MountingHole_2.5mm, MountingHole:MountingHole_2.5mm, F.Cu at (364.0, 171.9)
- SW1, SW10, SW12, SW13, SW14, SW15, SW16, SW17, SW18, SW19, SW20, SW21, SW22, SW23, SW24, SW25, SW26, SW27, SW28, SW29, SW30, SW31, SW32, SW33, SW34, SW35, SW36, SW37, SW38, SW39, SW4, SW40, SW41, SW42, SW43, SW44, SW45, SW46, SW47, SW48, SW49, SW5, SW50, SW51, SW52, SW53, SW54, SW55, SW56, SW57, SW6, SW7, SW8, SW9: footprint Button_Switch_Keyboard:SW_Cherry_MX1A_1.00u_Plate -> Button_Switch_Keyboard:SW_Cherry_MX_1.00u_PCB
- SW11: footprint Button_Switch_Keyboard:SW_Cherry_MX1A_1.00u_Plate -> Button_Switch_Keyboard:SW_Cherry_MX_6.25u_PCB
- SW2: footprint Button_Switch_Keyboard:SW_Cherry_MX1A_2.00u_Plate -> Button_Switch_Keyboard:SW_Cherry_MX_2.00u_PCB
- SW3, SW59: footprint Button_Switch_Keyboard:SW_Cherry_MX1A_1.50u_Plate -> Button_Switch_Keyboard:SW_Cherry_MX_1.50u_PCB
- SW58, SW61: footprint Button_Switch_Keyboard:SW_Cherry_MX1A_1.25u_Plate -> Button_Switch_Keyboard:SW_Cherry_MX_1.25u_PCB
- SW60, SW64: footprint Button_Switch_Keyboard:SW_Cherry_MX1A_1.75u_Plate -> Button_Switch_Keyboard:SW_Cherry_MX_1.75u_PCB
Connections:
- J1 pad 19: (no net) -> unconnected-(J1-Pad19)
Routing:
- net P11: track 450.8 -> 384.6 mm
- net P7: track 343.5 -> 277.4 mm, vias 0 -> 1
- net P2: track 294.4 -> 306.5 mm
- net P1: track 152.4 -> 162.0 mm
- net P4: track 297.2 -> 304.7 mm
- net P8: track 362.7 -> 369.2 mm
- net P6: track 280.3 -> 286.1 mm
- net WIRE_GND: track 116.6 -> 120.9 mm
- net P13: track 360.9 -> 356.9 mm
- net P12: track 393.7 -> 390.0 mm
- net P14: track 380.9 -> 377.3 mm
- net P5: track 302.1 -> 305.2 mm
- net P17: track 364.5 -> 367.0 mm
- net P3: track 153.3 -> 155.4 mm
- net BCS: track 381.5 -> 383.2 mm
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Other:
- net class Default removed
- board text added: "REV B"
- board text added: "Rev A: April 2021 by Ivo van Poorten Rev B: January 2022 Thomas Fleming"
- board text removed: "April 2021 by Ivo van Poorten"
- board text removed: "REV A"

Commit message: Add files via upload
Updated PCB to rev C. Moved backplane holes for better alignment. Moved main connector to prevent ribbon cable overlap with daughterboard.
Parts:
- moved J1 10.0 mm to (334.0, 70.0)
- moved REF12 1.35 mm to (183.3, 153.4)
- moved REF18 1.03 mm to (363.7, 170.9)
- moved REF15 0.50 mm to (342.5, 77.2)
- moved REF01 0.25 mm to (50.7, 77.4)
- moved REF02 0.25 mm to (129.3, 77.4)
- moved REF03 0.25 mm to (205.5, 77.4)
- moved REF04 0.25 mm to (262.7, 77.4)
- moved REF05 0.25 mm to (319.8, 77.4)
- moved REF09 0.25 mm to (317.6, 115.5)
Routing:
- net P12: track 390.0 -> 405.7 mm
- net P13: track 356.9 -> 372.1 mm
- net P14: track 377.3 -> 391.8 mm
- net P15: track 399.8 -> 413.8 mm
- net P11: track 384.6 -> 397.9 mm
- net OPTION: track 8.99 -> 21.7 mm
- net RESET: track 8.99 -> 21.7 mm
- net LED: track 14.1 -> 26.4 mm
- net START: track 8.99 -> 21.3 mm
- net P17: track 367.0 -> 379.0 mm
- net SELECT: track 8.99 -> 20.6 mm
- net GND: track 11.5 -> 22.8 mm
- net P16: track 406.8 -> 414.5 mm
- net P10: track 256.5 -> 263.4 mm
- net BCS: track 383.2 -> 376.5 mm
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Other:
- board text added: "REV C"
- board text added: "Rev C: April 2022 Thomas Fleming"
- board text removed: "REV B"
- board text removed: "Rev A: April 2021 by Ivo van Poorten Rev B: January 2022 Thomas Fleming"
